File: hardware/obj805.kicad_pcb (KiCad board)
At the start: 2 copper layers, 37 parts, among them J0 Conn_with_rapi, U1 l293d

Commit message: update
Parts:
- moved R500 186.4 mm to (31.4, 25.9)
- moved D_POWER1 186.4 mm to (25.3, 25.9)
- moved D_SVR1 169.3 mm to (24.0, 47.8)
- moved R100_2 166.3 mm to (22.4, 57.1), turned to 180 degrees
- moved D_MOTOR1 163.6 mm to (31.0, 57.4)
- moved R100_1 157.3 mm to (31.9, 48.7)
- moved R1 151.8 mm to (22.0, 36.2), turned to 180 degrees
- moved D_SYS1 151.7 mm to (28.0, 36.0)
- moved R3k1 139.2 mm to (68.1, 96.9)
- moved SW_UP1 139.2 mm to (72.8, 96.7)
- moved J_PWR1 123.0 mm to (176.1, 19.4), turned to 180 degrees
- moved R3k2 112.0 mm to (96.5, 116.2)
- moved SW_DOWN1 112.0 mm to (101.2, 111.3)
- moved UM_L1 104.6 mm to (243.3, 32.2)
- moved UM_H1 97.4 mm to (202.7, 32.5)
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Connections:
- D_SVR1 pad 1: Net-(D_SVR1-Pad1) -> Net-(D_POWER1-Pad1)
- D_SVR1 pad 2: Net-(D_POWER1-Pad1) -> Net-(D_SVR1-Pad2)
- J0 pad 6: Net-(J0-Pad6) -> Net-(D_POWER1-Pad1)
- R1 pad 2: Net-(J0-Pad6) -> Net-(D_POWER1-Pad1)
- R100_1 pad 1: Net-(D_SVR1-Pad1) -> Net-(D_SVR1-Pad2)
- R100_2 pad 2: Net-(J0-Pad6) -> Net-(D_POWER1-Pad1)
- U1 pad 4: Net-(J0-Pad6) -> Net-(D_POWER1-Pad1)
- U1 pad 5: Net-(J0-Pad6) -> Net-(D_POWER1-Pad1)
- U1 pad 6: Net-(J0-Pad6) -> Net-(D_POWER1-Pad1)
- U1 pad 7: Net-(J0-Pad6) -> Net-(D_POWER1-Pad1)
- UM_H1 pad 1: Net-(R3-Pad2) -> Net-(R6-Pad2)
- UM_H1 pad 13: Net-(J0-Pad6) -> Net-(D_POWER1-Pad1)
- UM_H1 pad 2: Net-(R4-Pad2) -> Net-(R5-Pad2)
- UM_H1 pad 3: Net-(R5-Pad2) -> Net-(R3-Pad2)
- UM_H1 pad 4: Net-(R6-Pad2) -> Net-(R4-Pad2)
- UM_H1 pad 5: Net-(R7-Pad2) -> Net-(R9-Pad2)
- UM_H1 pad 7: Net-(R9-Pad2) -> Net-(R7-Pad2)
- UM_L1 pad 1: Net-(R11-Pad2) -> Net-(R14-Pad2)
- UM_L1 pad 13: Net-(J0-Pad6) -> Net-(D_POWER1-Pad1)
- UM_L1 pad 2: Net-(R12-Pad2) -> Net-(R13-Pad2)
- UM_L1 pad 3: Net-(R13-Pad2) -> Net-(R11-Pad2)
- UM_L1 pad 4: Net-(R14-Pad2) -> Net-(R12-Pad2)
- UM_L1 pad 5: Net-(R15-Pad2) -> Net-(R17-Pad2)
- UM_L1 pad 7: Net-(R17-Pad2) -> Net-(R15-Pad2)
- U_H1 pad 3: Net-(J0-Pad6) -> Net-(D_POWER1-Pad1)
- U_H1 pad 8: Net-(J0-Pad6) -> Net-(D_POWER1-Pad1)
- U_L1 pad 3: Net-(J0-Pad6) -> Net-(D_POWER1-Pad1)
- U_L1 pad 8: Net-(J0-Pad6) -> Net-(D_POWER1-Pad1)
Routing:
- net Net-(D_POWER1-Pad1): track 0.00 -> 727.2 mm, vias 0 -> 4
- net Net-(J0-Pad1): track 0.00 -> 327.7 mm, vias 0 -> 6
- net Net-(J_PWR1-Pad1): track 0.00 -> 230.8 mm
- net Net-(J0-Pad22): track 0.00 -> 221.9 mm, vias 0 -> 4
- net Net-(J0-Pad18): track 0.00 -> 215.2 mm, vias 0 -> 6
- net Net-(D_MOTOR1-Pad2): track 0.00 -> 184.1 mm, vias 0 -> 4
- net Net-(D_SYS1-Pad2): track 0.00 -> 169.8 mm
- net Net-(J0-Pad16): track 0.00 -> 164.6 mm, vias 0 -> 5
- net Net-(J0-Pad13): track 0.00 -> 148.0 mm, vias 0 -> 1
- net Net-(J0-Pad11): track 0.00 -> 105.5 mm, vias 0 -> 1
- net Net-(J0-Pad2): track 0.00 -> 96.6 mm, vias 0 -> 3
- net Net-(J_MOTOR1-Pad1): track 0.00 -> 63.0 mm
- net Net-(R10-Pad2): track 0.00 -> 57.4 mm
- net GND: track 0.00 -> 50.5 mm, vias 0 -> 2
- net VCC: track 0.00 -> 42.8 mm, vias 0 -> 2
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- added copper zone on F.Cu, net Net-(D_POWER1-Pad1)

Commit message: update
Parts:
- added REF**: MountingHole_3mm, Mounting_Holes:MountingHole_3mm, F.Cu at (47.0, 28.0)
- U1: moved to B.Cu
- moved UM_L1 183.8 mm to (60.2, 48.0), turned to 90 degrees
- moved R17 176.3 mm to (74.4, 40.9), turned to 90 degrees
- moved R16 173.9 mm to (76.9, 40.9), turned to 90 degrees
- moved R15 171.6 mm to (79.4, 40.9), turned to 90 degrees
- moved R10 169.2 mm to (82.0, 40.9), turned to 90 degrees
- moved U_L1 163.0 mm to (80.7, 47.9), turned to 90 degrees
- moved R12 160.0 mm to (76.9, 54.7), turned to 270 degrees
- moved R11 157.3 mm to (79.5, 54.7), turned to 270 degrees
- moved R13 154.8 mm to (82.0, 54.7), turned to 270 degrees
- moved R14 152.3 mm to (84.5, 54.7), turned to 270 degrees
- moved UM_H1 147.8 mm to (60.2, 71.6), turned to 90 degrees
- moved R9 135.9 mm to (74.6, 64.4), turned to 90 degrees
- moved R8 133.0 mm to (77.2, 64.4), turned to 90 degrees
- moved R7 130.2 mm to (79.7, 64.4), turned to 90 degrees
- moved R2 127.6 mm to (82.1, 64.4), turned to 90 degrees
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Connections:
- D_POWER1 pad 1: Net-(D_POWER1-Pad1) -> GND
- D_SVR1 pad 1: Net-(D_POWER1-Pad1) -> GND
- J0 pad 6: Net-(D_POWER1-Pad1) -> GND
- J_MOTOR1 pad 2: Net-(D_POWER1-Pad1) -> GND
- J_PWR1 pad 2: Net-(D_POWER1-Pad1) -> GND
- J_PWR_J2 pad 2: Net-(D_POWER1-Pad1) -> GND
- J_PWR_J2 pad 3: Net-(D_POWER1-Pad1) -> GND
- R1 pad 2: Net-(D_POWER1-Pad1) -> GND
- R100_2 pad 2: Net-(D_POWER1-Pad1) -> GND
- R3k1 pad 1: Net-(D_POWER1-Pad1) -> GND
- R3k2 pad 1: Net-(D_POWER1-Pad1) -> GND
- U1 pad 14: Net-(D_POWER1-Pad1) -> GND
- U1 pad 15: Net-(D_POWER1-Pad1) -> GND
- U1 pad 16: Net-(D_POWER1-Pad1) -> GND
- U1 pad 17: Net-(D_POWER1-Pad1) -> GND
- U1 pad 4: Net-(D_POWER1-Pad1) -> GND
- U1 pad 5: Net-(D_POWER1-Pad1) -> GND
- U1 pad 6: Net-(D_POWER1-Pad1) -> GND
- U1 pad 7: Net-(D_POWER1-Pad1) -> GND
- UM_H1 pad 11: Net-(J0-Pad18) -> Net-(J0-Pad16)
- UM_H1 pad 12: Net-(J0-Pad22) -> Net-(J0-Pad18)
- UM_H1 pad 13: Net-(D_POWER1-Pad1) -> GND
- UM_H1 pad 14: Net-(J0-Pad16) -> Net-(J0-Pad22)
- UM_L1 pad 11: Net-(J0-Pad18) -> Net-(J0-Pad16)
- UM_L1 pad 12: Net-(J0-Pad22) -> Net-(J0-Pad18)
- UM_L1 pad 13: Net-(D_POWER1-Pad1) -> GND
- U_H1 pad 3: Net-(D_POWER1-Pad1) -> GND
- U_H1 pad 8: Net-(D_POWER1-Pad1) -> GND
- U_L1 pad 3: Net-(D_POWER1-Pad1) -> GND
- U_L1 pad 8: Net-(D_POWER1-Pad1) -> GND
Routing:
- net Net-(D_POWER1-Pad1): track 727.2 -> 0.00 mm, vias 4 -> 0
- net GND: track 50.5 -> 363.5 mm
- net Net-(J0-Pad22): track 221.9 -> 21.0 mm, vias 4 -> 0
- net Net-(J0-Pad18): track 215.2 -> 33.3 mm, vias 6 -> 0
- net Net-(J0-Pad1): track 327.7 -> 172.0 mm, vias 6 -> 0
- net Net-(D_MOTOR1-Pad2): track 184.1 -> 59.6 mm, vias 4 -> 1
- net Net-(J0-Pad16): track 164.6 -> 53.9 mm, vias 5 -> 0
- net Net-(J_PWR1-Pad1): track 230.8 -> 147.8 mm, vias 0 -> 1
- net Net-(D_SYS1-Pad2): track 169.8 -> 88.4 mm, vias 0 -> 1
- net Net-(J0-Pad13): track 148.0 -> 76.6 mm, vias 1 -> 0
- net Net-(J0-Pad11): track 105.5 -> 41.3 mm, vias 1 -> 0
- net Net-(J0-Pad15): track 14.4 -> 62.8 mm
- net Net-(J_MOTOR1-Pad1): track 63.0 -> 35.9 mm
- net Net-(R10-Pad2): track 57.4 -> 33.0 mm
- net VCC: track 42.8 -> 26.6 mm, vias 2 -> 0
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- added copper zone on B.Cu, net GND
- added copper zone on F.Cu, net GND
- removed copper zone on F.Cu, net Net-(D_POWER1-Pad1)
Other:
- net class Default: via_dia 0.6 -> 0.8; via_drill 0.4 -> 0.6
- net class power added: clearance 0.2, trace_width 0.75, via_dia 0.8, via_drill 0.6

Commit message: update;
Parts:
- removed the REF** at (47.0, 28.0)
- added REF**: MountingHole_2.7mm_M2.5, Mounting_Holes:MountingHole_2.7mm_M2.5, F.Cu at (24.0, 91.2)
- added REF**: MountingHole_2.7mm_M2.5, Mounting_Holes:MountingHole_2.7mm_M2.5, F.Cu at (82.0, 91.2)
- added REF**: MountingHole_2.7mm_M2.5, Mounting_Holes:MountingHole_2.7mm_M2.5, F.Cu at (82.0, 42.2)
- added REF**: MountingHole_2.7mm_M2.5, Mounting_Holes:MountingHole_2.7mm_M2.5, F.Cu at (24.0, 42.2)
- R10, R11, R12, R13, R14, R15, R16, R17, R2, R3, R4, R5, R6, R7, R8, R9, UM_H1, UM_L1: moved to B.Cu
- U1: moved to F.Cu
- moved R500 66.6 mm to (54.2, 82.5)
- moved D_POWER1 66.5 mm to (49.6, 82.5)
- moved R100_1 66.0 mm to (54.2, 88.7)
- moved D_SVR1 65.9 mm to (49.6, 88.7)
- moved D_SYS1 60.8 mm to (49.6, 79.5)
- moved R1 60.5 mm to (44.9, 79.5)
- moved D_MOTOR1 60.0 mm to (49.6, 85.7)
- moved R100_2 60.0 mm to (44.9, 85.7)
- moved R3k2 59.0 mm to (70.7, 88.8)
- moved R6 59.0 mm to (25.9, 73.1), turned to 180 degrees
- moved R3k1 58.5 mm to (58.8, 81.7), turned to 90 degrees
- moved SW_UP1 57.7 mm to (62.1, 80.8)
- moved R5 57.0 mm to (25.9, 70.5), turned to 180 degrees
- moved R3 54.8 mm to (25.9, 67.9), turned to 180 degrees
- moved R4 52.9 mm to (25.9, 65.4), turned to 180 degrees
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Connections:
- D_POWER1 pad 1: GND -> Net-(D_POWER1-Pad1)
- D_SVR1 pad 1: GND -> Net-(D_POWER1-Pad1)
- J0 pad 6: GND -> Net-(D_POWER1-Pad1)
- J_MOTOR1 pad 2: GND -> Net-(D_POWER1-Pad1)
- J_PWR1 pad 2: GND -> Net-(D_POWER1-Pad1)
- J_PWR_J2 pad 2: GND -> Net-(D_POWER1-Pad1)
- J_PWR_J2 pad 3: GND -> Net-(D_POWER1-Pad1)
- R1 pad 2: GND -> Net-(D_POWER1-Pad1)
- R100_2 pad 2: GND -> Net-(D_POWER1-Pad1)
- R3k1 pad 1: GND -> Net-(D_POWER1-Pad1)
- R3k2 pad 1: GND -> Net-(D_POWER1-Pad1)
- U1 pad 14: GND -> Net-(D_POWER1-Pad1)
- U1 pad 15: GND -> Net-(D_POWER1-Pad1)
- U1 pad 16: GND -> Net-(D_POWER1-Pad1)
- U1 pad 17: GND -> Net-(D_POWER1-Pad1)
- U1 pad 4: GND -> Net-(D_POWER1-Pad1)
- U1 pad 5: GND -> Net-(D_POWER1-Pad1)
- U1 pad 6: GND -> Net-(D_POWER1-Pad1)
- U1 pad 7: GND -> Net-(D_POWER1-Pad1)
- UM_H1 pad 1: Net-(R6-Pad2) -> Net-(R7-Pad2)
- UM_H1 pad 13: GND -> Net-(D_POWER1-Pad1)
- UM_H1 pad 2: Net-(R5-Pad2) -> Net-(R8-Pad2)
- UM_H1 pad 3: Net-(R3-Pad2) -> Net-(R9-Pad2)
- UM_H1 pad 5: Net-(R9-Pad2) -> Net-(R3-Pad2)
- UM_H1 pad 6: Net-(R8-Pad2) -> Net-(R5-Pad2)
- UM_H1 pad 7: Net-(R7-Pad2) -> Net-(R6-Pad2)
- UM_L1 pad 1: Net-(R14-Pad2) -> Net-(R15-Pad2)
- UM_L1 pad 13: GND -> Net-(D_POWER1-Pad1)
- UM_L1 pad 2: Net-(R13-Pad2) -> Net-(R16-Pad2)
- UM_L1 pad 3: Net-(R11-Pad2) -> Net-(R17-Pad2)
- UM_L1 pad 5: Net-(R17-Pad2) -> Net-(R11-Pad2)
- UM_L1 pad 6: Net-(R16-Pad2) -> Net-(R13-Pad2)
- UM_L1 pad 7: Net-(R15-Pad2) -> Net-(R14-Pad2)
- U_H1 pad 3: GND -> Net-(D_POWER1-Pad1)
- U_H1 pad 8: GND -> Net-(D_POWER1-Pad1)
- U_L1 pad 3: GND -> Net-(D_POWER1-Pad1)
- U_L1 pad 8: GND -> Net-(D_POWER1-Pad1)
Routing:
- net GND: track 363.5 -> 0.00 mm, vias 2 -> 0
- net Net-(J0-Pad1): track 172.0 -> 0.00 mm
- net Net-(J_PWR1-Pad1): track 147.8 -> 0.00 mm, vias 1 -> 0
- net Net-(J0-Pad2): track 97.5 -> 0.00 mm
- net Net-(D_SYS1-Pad2): track 88.4 -> 0.00 mm, vias 1 -> 0
- net Net-(J0-Pad13): track 76.6 -> 0.00 mm
- net Net-(J0-Pad15): track 62.8 -> 0.00 mm, vias 1 -> 0
- net Net-(D_MOTOR1-Pad2): track 59.6 -> 0.00 mm, vias 1 -> 0
- net Net-(J0-Pad16): track 53.9 -> 0.00 mm
- net Net-(R2-Pad2): track 53.1 -> 0.00 mm
- net Net-(J0-Pad11): track 41.3 -> 0.00 mm
- net Net-(J_MOTOR1-Pad1): track 35.9 -> 0.00 mm
- net Net-(J0-Pad18): track 33.3 -> 0.00 mm
- net Net-(R10-Pad2): track 33.0 -> 0.00 mm
- net VCC: track 26.6 -> 0.00 mm
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- removed copper zone on B.Cu, net GND
- removed copper zone on F.Cu, net GND
Other:
- board outline added: 65 x 56.5 mm
- net class Default: trace_width 0.25 -> 0.2

Commit message: update;
Parts:
- renumbered REF** to REF1, REF** to REF2, REF** to REF3, REF** to REF4
Changed lines of the file:
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@@
     (descr "Mounting Hole 2.7mm, no annular, M2.5")
     (tags "mounting hole 2.7mm no annular m2.5")
-    (fp_text reference REF** (at 0 -3.7) (layer F.SilkS)
+    (fp_text reference REF4 (at 0 -3.7) (layer F.SilkS)
       (effects (font (size 1 1) (thickness 0.15)))
     )
@@
     (descr "Mounting Hole 2.7mm, no annular, M2.5")
     (tags "mounting hole 2.7mm no annular m2.5")
-    (fp_text reference REF** (at 0 -3.7) (layer F.SilkS)
+    (fp_text reference REF3 (at 0 -3.7) (layer F.SilkS)
       (effects (font (size 1 1) (thickness 0.15)))
     )
@@
     (descr "Mounting Hole 2.7mm, no annular, M2.5")
     (tags "mounting hole 2.7mm no annular m2.5")
-    (fp_text reference REF** (at 0 -3.7) (layer F.SilkS)
+    (fp_text reference REF2 (at 0 -3.7) (layer F.SilkS)
       (effects (font (size 1 1) (thickness 0.15)))
     )
@@
     (descr "Mounting Hole 2.7mm, no annular, M2.5")
     (tags "mounting hole 2.7mm no annular m2.5")
-    (fp_text reference REF** (at 0 -3.7) (layer F.SilkS)
+    (fp_text reference REF1 (at 0 -3.7) (layer F.SilkS)
       (effects (font (size 1 1) (thickness 0.15)))
     )
