File: hardware/obj805.kicad_pcb (KiCad board)
At the start: 2 copper layers, 65 x 56.5 mm, 41 parts, among them J0 Conn_with_rapi, U1 l293d

Commit message: update
Routing:
- net Net-(D_POWER1-Pad1): track 0.00 -> 231.6 mm
- net Net-(J0-Pad1): track 0.00 -> 97.3 mm
- net Net-(J0-Pad13): track 0.00 -> 85.1 mm
- net Net-(J0-Pad15): track 0.00 -> 78.9 mm
- net Net-(D_MOTOR1-Pad2): track 0.00 -> 78.4 mm
- net Net-(J0-Pad11): track 0.00 -> 67.3 mm
- net Net-(D_SYS1-Pad2): track 0.00 -> 61.0 mm
- net Net-(J_PWR1-Pad1): track 0.00 -> 56.5 mm
- net Net-(J0-Pad2): track 0.00 -> 53.0 mm
- net Net-(J_MOTOR1-Pad1): track 0.00 -> 48.3 mm
- net Net-(J0-Pad22): track 0.00 -> 47.1 mm
- net Net-(R2-Pad2): track 0.00 -> 32.6 mm
- net Net-(J0-Pad18): track 0.00 -> 31.3 mm
- net Net-(UM_H1-Pad9): track 0.00 -> 29.4 mm
- net Net-(J0-Pad16): track 0.00 -> 28.5 mm
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
Commit message: update
Connections:
- D_POWER1 pad 1: Net-(D_POWER1-Pad1) -> GND
- D_SVR1 pad 1: Net-(D_POWER1-Pad1) -> GND
- J0 pad 6: Net-(D_POWER1-Pad1) -> GND
- J_MOTOR1 pad 2: Net-(D_POWER1-Pad1) -> GND
- J_PWR1 pad 2: Net-(D_POWER1-Pad1) -> GND
- J_PWR_J2 pad 2: Net-(D_POWER1-Pad1) -> GND
- J_PWR_J2 pad 3: Net-(D_POWER1-Pad1) -> GND
- R1 pad 2: Net-(D_POWER1-Pad1) -> GND
- R100_2 pad 2: Net-(D_POWER1-Pad1) -> GND
- R3k1 pad 1: Net-(D_POWER1-Pad1) -> GND
- R3k2 pad 1: Net-(D_POWER1-Pad1) -> GND
- U1 pad 14: Net-(D_POWER1-Pad1) -> GND
- U1 pad 15: Net-(D_POWER1-Pad1) -> GND
- U1 pad 16: Net-(D_POWER1-Pad1) -> GND
- U1 pad 17: Net-(D_POWER1-Pad1) -> GND
- U1 pad 4: Net-(D_POWER1-Pad1) -> GND
- U1 pad 5: Net-(D_POWER1-Pad1) -> GND
- U1 pad 6: Net-(D_POWER1-Pad1) -> GND
- U1 pad 7: Net-(D_POWER1-Pad1) -> GND
- UM_H1 pad 13: Net-(D_POWER1-Pad1) -> GND
- UM_L1 pad 13: Net-(D_POWER1-Pad1) -> GND
- U_H1 pad 3: Net-(D_POWER1-Pad1) -> GND
- U_H1 pad 8: Net-(D_POWER1-Pad1) -> GND
- U_L1 pad 3: Net-(D_POWER1-Pad1) -> GND
- U_L1 pad 8: Net-(D_POWER1-Pad1) -> GND
Routing:
- net GND: track 20.3 -> 308.2 mm
- net Net-(D_POWER1-Pad1): track 231.6 -> 0.00 mm
- net Net-(D_SYS1-Pad2): track 61.0 -> 67.8 mm
- net Net-(J0-Pad15): track 78.9 -> 85.1 mm
- net Net-(J0-Pad2): track 53.0 -> 55.6 mm
- net Net-(J_PWR1-Pad1): track 56.5 -> 58.9 mm
- net Net-(J0-Pad13): track 85.1 -> 86.9 mm
- net Net-(D_MOTOR1-Pad2): track 78.4 -> 80.0 mm
- net Net-(J_MOTOR1-Pad1): track 48.3 -> 49.5 mm
- added copper zone on B.Cu, net GND
- added copper zone on F.Cu, net GND

Commit message: update
Parts:
- removed D_MOTOR1, D_SYS1: LED, LEDs:LED_1206
- removed D_POWER1: LED_YELLOW, LEDs:LED_1206
- removed D_SVR1: LED_GREEN, LEDs:LED_1206
- removed J_MOTOR1, J_PWR1: Conn_01x02, Pin_Headers:Pin_Header_Straight_1x02_Pitch2.54mm
- removed J_PWR_J2: Jack-DC, Connectors:JACK_ALIM
- removed R1, R10, R100_1, R100_2, R11, R12, R13, R14, R15, R16, R17, R2, R3, R3k1, R3k2, R4, R5, R500, R6, R7, R8, R9: R, Resistors_SMD:R_0805
- removed SW_DOWN1, SW_UP1: SW_Push, Buttons_Switches_THT:SW_PUSH_6mm
- removed UM_H1, UM_L1: 74HC595, SMD_Packages:SO-16-N
- removed U_H1, U_L1: 7SEGMENT_CC, l293d:7SegmentLED_3611
- added F0: Conn_01x02, Pin_Headers:Pin_Header_Straight_1x02_Pitch2.54mm, F.Cu at (115.2, 90.4)
- added P0: Jack-DC, Connectors:JACK_ALIM, F.Cu at (112.9, 78.9)
- U1: value l293d -> L293D; footprint l293d:SOIC-20 -> l293d:L293D; moved to B.Cu
- moved J0 84.1 mm to (110.9, 61.9)
- moved REF1 84.0 mm to (106.0, 60.6)
- moved REF2 84.0 mm to (164.0, 60.6)
- moved REF3 84.0 mm to (164.0, 109.7)
- moved REF4 84.0 mm to (106.0, 109.7)
- moved U1 77.8 mm to (147.2, 75.1), turned to 0 degrees
Connections:
- J0 pad 12: Net-(D_MOTOR1-Pad2) -> Net-(J0-Pad12)
- J0 pad 14: Net-(J0-Pad14) -> Net-(F0-Pad2)
- J0 pad 20: Net-(J0-Pad20) -> Net-(F0-Pad2)
- J0 pad 25: Net-(J0-Pad25) -> Net-(F0-Pad2)
- J0 pad 30: Net-(J0-Pad30) -> Net-(F0-Pad2)
- J0 pad 34: Net-(J0-Pad34) -> Net-(F0-Pad2)
- J0 pad 39: Net-(J0-Pad39) -> Net-(F0-Pad2)
- J0 pad 4: Net-(J0-Pad4) -> Net-(J0-Pad2)
- J0 pad 6: GND -> Net-(F0-Pad2)
- J0 pad 9: Net-(J0-Pad9) -> Net-(F0-Pad2)
- U1 pad 12: Net-(U1-Pad12) -> Net-(F0-Pad2)
- U1 pad 13: Net-(U1-Pad13) -> Net-(F0-Pad2)
- U1 pad 14: GND -> Net-(U1-Pad14)
- U1 pad 15: GND -> Net-(U1-Pad15)
- U1 pad 16: GND -> Net-(J0-Pad2)
- U1 pad 2: Net-(D_MOTOR1-Pad2) -> Net-(J0-Pad35)
- U1 pad 4: GND -> Net-(F0-Pad2)
- U1 pad 5: GND -> Net-(F0-Pad2)
- U1 pad 6: GND -> Net-(U1-Pad6)
- U1 pad 7: GND -> Net-(U1-Pad7)
Routing:
- net GND: track 308.2 -> 0.00 mm
- net Net-(F0-Pad2): track 0.00 -> 144.7 mm
- net Net-(P0-Pad1): track 0.00 -> 117.7 mm
- net Net-(J0-Pad1): track 97.3 -> 0.00 mm
- net Net-(J0-Pad13): track 86.9 -> 0.00 mm
- net Net-(J0-Pad15): track 85.1 -> 0.00 mm
- net Net-(D_MOTOR1-Pad2): track 80.0 -> 0.00 mm
- net Net-(J0-Pad11): track 67.1 -> 0.00 mm
- net Net-(U1-Pad10): track 58.9 -> 0.00 mm
- net Net-(J0-Pad22): track 47.1 -> 0.00 mm
- net Net-(J0-Pad7): track 67.8 -> 27.6 mm
- net Net-(F0-Pad1): track 49.5 -> 85.2 mm
- net Net-(J0-Pad2): track 55.6 -> 91.2 mm
- net Net-(R2-Pad2): track 32.6 -> 0.00 mm
- net Net-(J0-Pad18): track 31.2 -> 0.00 mm
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- added copper zone on F.Cu, net Net-(F0-Pad2)
- removed copper zone on B.Cu, net GND
- removed copper zone on F.Cu, net GND
Other:
- net class Default: clearance 0.2 -> 0.4; trace_width 0.2 -> 0.5
- net class power: clearance 0.2 -> 0.5; trace_width 0.75 -> 1
- rule trace_clearance: 0.2 -> 0.4

Commit message: update
Parts:
- U1: moved to F.Cu
Routing:
- net Net-(F0-Pad2): track 144.7 -> 44.9 mm
- net Net-(F0-Pad1): track 85.2 -> 34.0 mm
- net Net-(J0-Pad2): track 91.2 -> 40.6 mm
- net Net-(J0-Pad35): track 21.2 -> 62.5 mm
- net Net-(P0-Pad1): track 117.7 -> 79.5 mm
- net Net-(J0-Pad7): track 27.6 -> 33.7 mm
- added copper zone on B.Cu, net Net-(F0-Pad2)

Commit message: update;
Routing:
- net Net-(J0-Pad35): track 62.5 -> 126.5 mm
- net Net-(F0-Pad2): track 44.9 -> 34.1 mm
- net Net-(J0-Pad7): track 33.7 -> 37.4 mm
